File: __module_interface.sch (KiCad schematic (older format))
At the start: 32 parts, among them J10 exp FM, J11 tri_out, J12 saw_out, J13 squ_out, J14 bus_L, J15 bus_R, J6 lin FM, J7 sync, J8 V/oct_1, J9 V/oct_2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

Commit message: Artworks on pcbs are done.
Parts:
- R39: footprint Resistor_THT:R_Axial_DIN0207_L6.3mm_D2.5mm_P2.54mm_Vertical -> Resistor_THT:R_Axial_DIN0207_L6.3mm_D2.5mm_P7.62mm_Horizontal
Changed lines of the file:
@@
 $Descr A4 11693 8268
 encoding utf-8
-Sheet 3 3
+Sheet 2 2
 Title ""
 Date ""
@@
 F 0 "R39" V 8693 4000 50  0000 C CNN
 F 1 "3k" V 8784 4000 50  0000 C CNN
-F 2 "Resistor_THT:R_Axial_DIN0207_L6.3mm_D2.5mm_P2.54mm_Vertical" V 8830 4000 50  0001 C CNN
+F 2 "Resistor_THT:R_Axial_DIN0207_L6.3mm_D2.5mm_P7.62mm_Horizontal" V 8830 4000 50  0001 C CNN
 F 3 "~" H 8900 4000 50  0001 C CNN
 	1    8900 4000
