File: 2131VCO.kicad_pcb (KiCad board)
At the start: 2 copper layers, 76.2 x 99.1 mm, 104 parts, among them J1 Vref, J10 exp FM, J11 tri_out, J12 saw_out, J13 squ_out, J14 bus_L, J15 bus_R, J2 bus_L, J3 tri, J4 bus_R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

Commit message: Fixed a minor problem; - position of HF_track and init_freq trimmers - marking in the front panel
Parts:
- moved C11 12.8 mm to (137.2, 124.5)
- moved C9 12.8 mm to (137.2, 115.6)
- moved R14 12.8 mm to (137.2, 119.4)
- moved R26 12.8 mm to (115.6, 130.8)
- moved R8 12.8 mm to (119.4, 83.8)
- moved D2 12.8 mm to (137.2, 108.0)
- moved J4 12.8 mm to (137.2, 132.1)
- moved R11 12.8 mm to (119.4, 95.2)
- moved R12 12.8 mm to (129.5, 81.3)
- moved R23 12.8 mm to (115.6, 128.3)
- moved R31 12.8 mm to (115.6, 138.4)
- moved REF** 12.8 mm to (135.9, 76.2)
- moved RV4 12.8 mm to (119.4, 120.7)
- moved U2 12.8 mm to (119.4, 111.8)
- moved C5 12.8 mm to (121.9, 115.6)
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