File: ModuleCore.kicad_pcb (KiCad board)
At the start: 2 copper layers, 38.1 x 99.1 mm, 70 parts, among them J1 Vref, J2 bus_L, J3 tri, J4 bus_R, J5 power_bus, U1 TL074, U2 L78L05_TO92, U3 L79L05_TO92, U4 SSI2131, U5 LM317L_TO92

Commit message: Fixed a minor problem; - position of HF_track and init_freq trimmers - marking in the front panel
Parts:
- moved C15 2.84 mm to (108.0, 86.4)
- moved R17 2.54 mm to (88.9, 54.6)
- moved R3 2.54 mm to (88.9, 62.2)
- moved RV1 1.27 mm to (85.1, 58.4)
- moved RV3 1.27 mm to (85.1, 53.3)
Routing:
- net +5V: track 53.9 -> 51.2 mm
- net Net-(R10-Pad2): track 49.0 -> 51.5 mm
- net Net-(RV3-Pad3): track 42.4 -> 41.1 mm
- net Net-(R3-Pad2): track 5.61 -> 6.88 mm
- net Net-(R17-Pad1): track 5.61 -> 6.88 mm
Other:
- board text added: "2131VCO ver. 2"
- board text removed: "2131VCO ver. 1"
